File: kicad/lucy.kicad_pcb (KiCad board)
At the start: 2 copper layers, 96 x 56 mm, 63 parts, among them J1 Channel1, J10 Channel7, J11 Channel8, J2 Debug, J3 on/off, J4 Channel2, J5 USB-C, J6 Channel3, J7 Channel4, J8 Channel5, J9 Channel6, Q2 AO3400A, U1 TMUX1208, U3 STM32L062K8Tx, U4 TPS7A2-3.0, U5 RFM96W-433, U7 TP4056, U8 SRV05-4

Commit message: lucy_v1.0
Connections:
- J2 pad 9: pb5 -> GND
- U3 pad 28: pb5 -> mux_data
Routing:
- net mux_data: track 13.1 -> 26.1 mm, vias 0 -> 2
- net pb5: track 6.01 -> 0.00 mm
Other:
- board text removed: "pb5"
